File: board/scopeboy.kicad_sch (KiCad schematic)
At the start: 94 parts, among them J1 USB_B_Micro, J2 Conn_02x26_Odd_Even, J3 SM03B-SRSS-TB, J4 SM03B-SRSS-TB, J5 Conn_02x26_Odd_Even, J6 Conn_01x10, J7 SM04B-SRSS-TB, J8 HDMI_A, SW1 SW_Push, SW2 SW_Push, SW3 RotaryEncoder_Switch, U1 W25Q128JVS, U2 DNF, U3 NCP1117-3.3_SOT223, U4 RP2350_80QFN, U5 LP2985-3.3, U6 LM27762, U7 ADC08060, Y1 ABM8-272-T3

Commit message: More work on front end circuit, and GPIO connections
Parts:
- removed J1: USB_B_Micro, Connector_USB:USB_Micro-B_Amphenol_10103594-0001LF_Horizontal, symbol Connector:USB_B_Micro
- removed J2, J5: Conn_02x26_Odd_Even, Connector_PinHeader_2.54mm:PinHeader_2x26_P2.54mm_Vertical, symbol Connector_Generic:Conn_02x26_Odd_Even
- added J2: USB_C_Receptacle_USB2.0_16P, Connector_USB:USB_C_Receptacle_GCT_USB4105-xx-A_16P_TopMnt_Horizontal, symbol Connector:USB_C_Receptacle_USB2.0_16P
- added R46, R47: 5.1k, Resistor_SMD:R_1206_3216Metric, symbol Device:R
Connections:
- net +3V3Pico is gone; now on net +3V3: J6.2 (Pin_2), J7.2 (Pin_2)
- net GPIO1 is gone; now on net LCDCS: U4.78 (GPIO1)
- net GPIO10 is gone; now on net D2: U4.8 (GPIO10)
- net GPIO11 is gone; now on net D3: U4.9 (GPIO11)
- net GPIO2 is gone; now on net SCK: U4.79 (GPIO2)
- net GPIO20 is gone; now on net SDA: U4.20 (GPIO20)
- net GPIO21 is gone; now on net SCL: U4.21 (GPIO21)
- net GPIO23 is gone; now on net ROTCLK: U4.23 (GPIO23)
- net GPIO24 is gone; now on net ROTDT: U4.25 (GPIO24)
- net GPIO25 is gone; now on net ROTSW: U4.26 (GPIO25)
- net GPIO28 is gone; now on net TX: U4.36 (GPIO28)
- net GPIO29 is gone; now on net RX: U4.37 (GPIO29)
- net GPIO3 is gone; now on net MISO: U4.80 (GPIO3)
- net GPIO8 is gone; now on net D0: U4.6 (GPIO8)
- net GPIO9 is gone; now on net D1: U4.7 (GPIO9)
- net D4: now also U4.11 (GPIO12)
- net D5: now also U4.12 (GPIO13)
- net D6: now also U4.13 (GPIO14)
- net D7: now also U4.14 (GPIO15)
- net GND: now also J2.A1 (GND), J2.A12 (GND), J2.B1 (GND), J2.B12 (GND), R46.1, R47.1
- net GPIO0: no longer U4.77 (GPIO0)
- net GPIO12: no longer U4.11 (GPIO12)
- net GPIO13: no longer U4.12 (GPIO13)
- net GPIO14: no longer U4.13 (GPIO14)
- net GPIO15: no longer U4.14 (GPIO15)
- net MOSI: now also U4.77 (GPIO0)
- net USB_D+: now also J2.A6 (D+), J2.B6 (D+)
- net USB_D-: now also J2.A7 (D-), J2.B7 (D-)
- net VBUS: now also J2.A4 (VBUS), J2.A9 (VBUS), J2.B4 (VBUS), J2.B9 (VBUS)
- net BACKLIGHT renamed Backlight
- net RESET renamed Reset
- new net: J2.B5 (CC2), R47.2
- new net: J2.A5 (CC1), R46.2
- no-connect marks 1 -> 0
Other:
- sheet Analog Front End ports: added SEL0, SEL1; removed none
- note added: "Analog Front End"
- note added: "I picked these pins at random. Move if needed"
- note added: "TODO CHANGE THESE TO BATTERY VOLTAGES"
- note added: "TODO connect all the GPIO pins"
- note added: "TODO figure out how to handle the SD Card"
- note added: "TODO place SEL pins"
- note added: "TODO place chassis pins"
- note added: "USB Port"
- note removed: "IOs"
- note removed: "TODO check if this needs to be 5V"
- note removed: "TODO delete these headers"
- note removed: "TODO swap this for USB-C"
- moved on the sheet: C1, C6, U3

Commit message: All components in layout
Parts:
- H1, H2, H3, H4: footprint MountingHole:MountingHole_2.7mm_M2.5 -> MountingHole:MountingHole_3.2mm_M3_Pad_TopBottom; now left out of the parts list
- renumbered C2 to C1, C3 to C2, C4 to C3, C5 to C4, C7 to C5, C1 to C6, C8 to C7, C9 to C8, C6 to C9, J2 to J1, J3 to J2, J4 to J3, J6 to J4, J7 to J5, J8 to J6, R8 to R10, R9 to R11, R10 to R12, R11 to R13, R12 to R14, R13 to R15, R14 to R16, R15 to R17, R16 to R18, R17 to R19, R18 to R20, R19 to R21, R20 to R22, R21 to R23, R22 to R24, R23 to R25, R24 to R26, R25 to R27, R26 to R28, R27 to R29, R28 to R30, R29 to R31, R30 to R32, R46 to R6, R47 to R7, R6 to R8, R7 to R9
